Commit message: add launc file

File: urdf/robot.urdf.xacro (robot description, xacro)
@@ -8,5 +8,5 @@
         <color rgba="0.0 0.0 0.8 1"/>
     </material>
-    <material name="black">
+    <material name="red">
         <color rgba="0.8 0.0 0.0 1"/>
     </material>
@@ -74,5 +74,5 @@
                 <box size="0.05 0.05 0.05"/>
             </geometry>
-            <material name="black"/>
+            <material name="red"/>
         </visual>
         <collision>
@@ -89,23 +89,24 @@
     <!-- Gazebo Differential Drive Plugin -->
     <gazebo>
-        <plugin name="diff_drive" filename="libgazebo_ros_diff_drive.so">
+        <plugin filename="gz-sim-diff-drive-system" name="gz::sim::systems::DiffDrive">
             <!-- Wheel Information -->
             <left_joint>front_left_wheel_joint</left_joint>
             <right_joint>front_right_wheel_joint</right_joint>
+            <left_joint>rear_left_wheel_joint</left_joint>
+            <right_joint>rear_right_wheel_joint</right_joint>
             <!-- Kinematics -->
             <wheel_separation>0.36</wheel_separation>
-            <wheel_diameter>0.2</wheel_diameter>
+            <wheel_reduis>0.1</wheel_reduis>
             <!-- Limits -->
             <max_wheel_torque>20</max_wheel_torque>
             <max_wheel_acceleration>1.0</max_wheel_acceleration>
             <!-- Output -->
-            <odometry_frame>odom</odometry_frame>
-            <robot_base_frame>base_footprint</robot_base_frame>
-            <publish_odom>true</publish_odom>
-            <publish_odom_tf>true</publish_odom_tf>
-            <publish_wheel_tf>true</publish_wheel_tf>
-            <!-- Topic to subscribe to -->
-            <command_topic>cmd_vel</command_topic>
+            <topic>cmd_vel</topic>
+            <odom_topic>odom</odom_topic>
+            <frame_id>odom</frame_id>
+            <child_frame_id>base_footprint</child_frame_id>
+            <odom_publisher_frequency>30</odom_publisher_frequency>
         </plugin>
+        <plugin filename="gz-sim-joint-state-publisher-system" name="gz::sim::systems::JointStatePublisher"/>
     </gazebo>
 </robot>
